File: hardware/filter.sch (KiCad schematic (older format))
At the start: 14 parts, among them U2 SKY13322-375LF, U3 LP0603, U4 LP0603, U5 5515LP15A730, U6 3550LP14A300, U7 SKY13322-375LF

Commit message: updated csv file
Parts:
- U4: value LP0603 -> LP06031880
Changed lines of the file:
@@
 P 5500 1100
 F 0 "U4" H 5525 1437 60  0000 C CNN
-F 1 "LP0603" H 5525 1331 60  0000 C CNN
+F 1 "LP06031880" H 5525 1331 60  0000 C CNN
 F 2 "violet:LP0603A0902" H 5600 850 60  0001 C CNN
 F 3 "" H 5600 850 60  0000 C CNN
